Commit message: Add cable mass to Solo12 URDF.

File: robots/solo_description/robots/solo12.urdf (robot description, URDF)
Before this commit: robot solo, 17 links, 16 joints
Links:
- added link cables, mass 0.15
Joints:
- added joint cable_mass_joint: type fixed, parent base_link, child cables, origin xyz=-0.20 0.0 0.0 rpy=0 0 0
